File: kicad project/tascamusbc.kicad_sch (KiCad schematic)
At the start: 4 parts, among them J1 USB_B_Mini, J2 USB_C_Receptacle_USB2.0

Commit message: updated project
Connections:
- net CC2: now reaches J2.B5 (CC2), R2.1
- net GND: now reaches J1.5 (GND), J2.A1 (GND), J2.A12 (GND), J2.B1 (GND), J2.B12 (GND), R1.2, R2.2
- net CC1: now reaches J2.A5 (CC1), R1.1
- net VBUS: now reaches J1.1 (VBUS), J2.A4 (VBUS), J2.A9 (VBUS), J2.B4 (VBUS), J2.B9 (VBUS)
- net D-: now reaches J1.2 (D-), J2.A7 (D-), J2.B7 (D-)
- net D+: now reaches J1.3 (D+), J2.A6 (D+), J2.B6 (D+)
- net SHIELD: now reaches J1.6 (Shield), J2.S1 (SHIELD)
- no-connect marks 1 -> 3
Other:
- moved on the sheet: R1, R2
Changed lines of the file:
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@@
   (junction (at 100.33 57.15) (diameter 0) (color 0 0 0 0)
   )
-  (junction (at 107.95 50.8) (diameter 0) (color 0 0 0 0)
+  (junction (at 115.57 81.28) (diameter 0) (color 0 0 0 0)
   )
-  (junction (at 107.95 81.28) (diameter 0) (color 0 0 0 0)
+  (junction (at 115.57 50.8) (diameter 0) (color 0 0 0 0)
   )
   (no_connect (at 121.92 53.34))
-  (wire (pts (xy 107.95 50.8) (xy 107.95 81.28))
+  (no_connect (at 100.33 71.12))
+  (no_connect (at 100.33 73.66))
+  (wire (pts (xy 107.95 48.26) (xy 100.33 48.26))
     (stroke (width 0) (type default))
   )
-  (wire (pts (xy 107.95 48.26) (xy 107.95 50.8))
+  (wire (pts (xy 115.57 50.8) (xy 115.57 81.28))
+    (stroke (width 0) (type default))
+  )
+  (wire (pts (xy 115.57 48.26) (xy 115.57 50.8))
     (stroke (width 0) (type default))
   )
   (wire (pts (xy 118.11 48.26) (xy 121.92 48.26))
+    (stroke (width 0) (type default))
+  )
+  (wire (pts (xy 115.57 81.28) (xy 129.54 81.28))
+    (stroke (width 0) (type default))
+  )
+  (wire (pts (xy 107.95 50.8) (xy 100.33 50.8))
     (stroke (width 0) (type default))
   )
@@
     (stroke (width 0) (type default))
   )
-  (wire (pts (xy 107.95 81.28) (xy 129.54 81.28))
-    (stroke (width 0) (type default))
-  )
   (wire (pts (xy 120.65 57.15) (xy 120.65 50.8))
     (stroke (width 0) (type default))
@@
   )
   (wire (pts (xy 77.47 83.82) (xy 77.47 81.28))
+    (stroke (width 0) (type default))
+  )
+  (wire (pts (xy 85.09 81.28) (xy 115.57 81.28))
     (stroke (width 0) (type default))
   )
@@
     (stroke (width 0) (type default))
   )
-  (wire (pts (xy 85.09 81.28) (xy 107.95 81.28))
-    (stroke (width 0) (type default))
-  )
   (wire (pts (xy 100.33 62.23) (xy 118.11 62.23))
     (stroke (width 0) (type default))
@@
     (stroke (width 0) (type default))
   )
-  (symbol (lib_id "Device:R") (at 104.14 50.8 90) (unit 1)
+  (label "CC2" (at 101.6 50.8 0) (fields_autoplaced)
+    (effects (font (size 1.27 1.27)) (justify left bottom))
+  )
+  (label "CC1" (at 101.6 48.26 0) (fields_autoplaced)
+    (effects (font (size 1.27 1.27)) (justify left bottom))
+  )
+  (label "VBUS" (at 107.95 43.18 0) (fields_autoplaced)
+    (effects (font (size 1.27 1.27)) (justify left bottom))
+  )
+  (label "D+" (at 101.6 62.23 0) (fields_autoplaced)
+    (effects (font (size 1.27 1.27)) (justify left bottom))
+  )
+  (label "GND" (at 115.57 81.28 0) (fields_autoplaced)
+    (effects (font (size 1.27 1.27)) (justify left bottom))
+  )
+  (label "D-" (at 101.6 57.15 0) (fields_autoplaced)
+    (effects (font (size 1.27 1.27)) (justify left bottom))
+  )
+  (label "SHIELD" (at 113.03 83.82 0) (fields_autoplaced)
+    (effects (font (size 1.27 1.27)) (justify left bottom))
+  )
+  (symbol (lib_id "Device:R") (at 111.76 50.8 90) (unit 1)
     (in_bom yes) (on_board yes) (dnp no)
-    (property "Reference" "R2" (at 110.49 50.8 90)
+    (property "Reference" "R2" (at 111.76 45.72 90)
       (effects (font (size 1.27 1.27)))
     )
-    (property "Value" "5.1K" (at 114.3 50.8 90)
-      (effects (font (size 1.27 1.27)))
-    )
-    (property "Footprint" "Resistor_SMD:R_0402_1005Metric_Pad0.72x0.64mm_HandSolder" (at 104.14 52.578 90)
+    (property "Value" "5.1K" (at 113.03 53.34 90)
       (effects (font (size 1.27 1.27)) hide)
     )
-    (property "Datasheet" "~" (at 104.14 50.8 0)
+    (property "Footprint" "Resistor_SMD:R_0402_1005Metric_Pad0.72x0.64mm_HandSolder" (at 111.76 52.578 90)
+      (effects (font (size 1.27 1.27)) hide)
+    )
+    (property "Datasheet" "~" (at 111.76 50.8 0)
       (effects (font (size 1.27 1.27)) hide)
     )
@@
     )
   )
-  (symbol (lib_id "Device:R") (at 104.14 48.26 90) (unit 1)
+  (symbol (lib_id "Device:R") (at 111.76 48.26 90) (unit 1)
     (in_bom yes) (on_board yes) (dnp no)
-    (property "Reference" "R1" (at 110.49 48.26 90)
+    (property "Reference" "R1" (at 109.22 45.72 90)
       (effects (font (size 1.27 1.27)))
     )
-    (property "Value" "5.1K" (at 114.3 48.26 90)
+    (property "Value" "5.1K" (at 115.57 45.72 90)
       (effects (font (size 1.27 1.27)))
     )
-    (property "Footprint" "Resistor_SMD:R_0402_1005Metric_Pad0.72x0.64mm_HandSolder" (at 104.14 50.038 90)
+    (property "Footprint" "Resistor_SMD:R_0402_1005Metric_Pad0.72x0.64mm_HandSolder" (at 111.76 50.038 90)
       (effects (font (size 1.27 1.27)) hide)
     )
-    (property "Datasheet" "~" (at 104.14 48.26 0)
+    (property "Datasheet" "~" (at 111.76 48.26 0)
       (effects (font (size 1.27 1.27)) hide)
     )
