File: kicad project/tascamusbc.kicad_pcb (KiCad board)
At the start: 2 copper layers, 8.6 x 9.2 mm, 4 parts, among them J1 USB_B_Mini, J2 USB_C_Receptacle_USB2.0

Commit message: updated project
Parts:
- J1: moved to F.Cu
- moved R1 0.10 mm to (67.2, 73.8)
- moved R2 0.10 mm to (61.6, 73.8)
- turned J1 to 180 degrees
Connections:
- net Net-(J1-D+) renamed /D+
- net Net-(J1-D-) renamed /D-
- net Net-(J1-GND) renamed /GND
- net Net-(J1-VBUS) renamed /VBUS
- net Net-(J2-CC1) renamed /CC1
- net Net-(J2-CC2) renamed /CC2
- J1 pad 4: (no net) -> unconnected-(J1-ID-Pad4)
- J2 pad A8: (no net) -> unconnected-(J2-SBU1-PadA8)
- J2 pad B8: (no net) -> unconnected-(J2-SBU2-PadB8)
- J2 pad S1: (no net) -> /SHIELD
Routing:
- net /SHIELD: track 0.00 -> 19.6 mm
- net /D-: track 6.05 -> 4.26 mm, vias 1 -> 0
Other:
- board text added: ":p"
- board text added: "TSCM DR-40 USB-C V1.2 by sable"
- board text removed: "TSCM DR-40 USB-C V1.1 Stevano"

Commit message: updated schematic
Parts:
- moved J1 0.07 mm to (64.4, 72.3)
Routing:
- net /SHIELD: track 19.6 -> 1.95 mm
- net /GND: track 20.1 -> 19.4 mm
- added copper zone on B.Cu, net /SHIELD
- added copper zone on F.Cu, net /SHIELD
Other:
- board text added: "TSCM DR-40 USB-C V1.3 by sable"
- board text added: "who needs clearences, lol?"
- board text removed: "TSCM DR-40 USB-C V1.2 by sable"
- board text removed: "hopefully i'm only seen once"
